Commit message: Kapsamli guvenlik+performans: emergency status kanalindan da, guvenli iptal (dikey kalkis+kesintisiz koridor), STOP destegi, disk collision kaldirildi (RTF), 60sn demo modu

File: src/end_effector_ros2/urdf/robot_with_sander.urdf.xacro (robot description, xacro)
@@ -86,5 +86,5 @@
       <origin xyz="0 0 0" rpy="0 0 0"/>
       <geometry>
-        <cylinder radius="0.045" length="0.02"/>
+        <cylinder radius="0.001" length="0.001"/>
       </geometry>
       <material name="sander_pad_red">
@@ -105,5 +105,5 @@
       <origin xyz="0 0 0" rpy="0 0 0"/>
       <geometry>
-        <cylinder radius="0.045" length="0.02"/>
+        <cylinder radius="0.001" length="0.001"/>
       </geometry>
     </collision>

Commit message: Kirmizi disk gorseli geri, emergency kenar-tetik (park dongusu bug), hizli acil geri cekilme, parkta() korumasi

File: src/end_effector_ros2/urdf/robot_with_sander.urdf.xacro (robot description, xacro)
@@ -86,5 +86,5 @@
       <origin xyz="0 0 0" rpy="0 0 0"/>
       <geometry>
-        <cylinder radius="0.001" length="0.001"/>
+        <cylinder radius="0.045" length="0.02"/>
       </geometry>
       <material name="sander_pad_red">

Commit message: SPEC: STOP=oldugu yerde dur (park yok), EMERGENCY=dur+park; zimpara min 5cm pas; zimpara GOVDE carpisma kutusu kucultuldu (disk esige inebiliyor)

File: src/end_effector_ros2/urdf/robot_with_sander.urdf.xacro (robot description, xacro)
@@ -67,5 +67,5 @@
       <origin xyz="0.003 -0.055 0.105" rpy="0 0 0"/>
       <geometry>
-        <box size="0.17 0.30 0.20"/>
+        <box size="0.05 0.05 0.05"/>
       </geometry>
     </collision>
